Commit message: much better odometry (closer to reality)

File: urdf/macros.xacro (robot description, xacro)
@@ -16,5 +16,5 @@
                 <origin xyz="0 0 0" rpy="0 ${PI/2} ${PI/2}"/>
                 <geometry>
-                    <cylinder length="${wheelWidth}" radius="${wheelRadius}"/>
+                     <sphere radius="${wheelRadius}" />
                 </geometry>
             </collision>
@@ -88,6 +88,6 @@
         </joint>
         <gazebo reference="${name}">
-            <mu1>0.01</mu1>
-            <mu2>0.01</mu2>
+            <mu1>0.0</mu1>
+            <mu2>0.0</mu2>
             <material>Gazebo/Red</material>
         </gazebo>
