Commit message: options for localisation stress-test

File: urdf/macros.xacro (robot description, xacro)
@@ -16,5 +16,8 @@
                 <origin xyz="0 0 0" rpy="0 ${PI/2} ${PI/2}"/>
                 <geometry>
-                     <sphere radius="${wheelRadius}" />
+                    <!-- Good odometry, more realistic -->
+                    <sphere radius="${wheelRadius}" />
+                    <!-- Bad odometry, stress-test for localisation -->
+                    <!--<cylinder length="${wheelWidth}" radius="${wheelRadius}"/>-->
                 </geometry>
             </collision>
@@ -88,6 +91,6 @@
         </joint>
         <gazebo reference="${name}">
-            <mu1>0.0</mu1>
-            <mu2>0.0</mu2>
+            <mu1>0.01</mu1>
+            <mu2>0.01</mu2>
             <material>Gazebo/Red</material>
         </gazebo>
