Commit message: use tim for obstacles

File: urdf/krabby.xacro (robot description, xacro)
@@ -15,5 +15,8 @@
   <xacro:property name="cameraSize" value="0.05"/>
   <xacro:property name="cameraMass" value="0.1"/>
-  <xacro:property name="lidarZPos" value="0.250"/>
+  <xacro:property name="lidarZPos" value="0.3"/>
+  <!-- mapping
+    <xacro:property name="lidarZPos" value="0.06"/>
+  -->
   <xacro:property name="lidarMass" value="0.1"/>
   <xacro:property name="lidarRadius" value="0.05"/>
@@ -118,5 +121,5 @@
   </link>
   <joint name="neato_laser" type="fixed">
-    <origin xyz="0 0 ${lidarZPos}" rpy="0 0 0"/>
+    <origin xyz="0 0 ${lidarZPos}" rpy="3.14159 0 0"/>
     <parent link="chassis"/>
     <child link="neato_laser"/>

Commit message: tim top

File: urdf/krabby.xacro (robot description, xacro)
@@ -100,5 +100,5 @@
     <child link="camera_link"/>
   </joint>
-  <link name="neato_laser">
+  <link name="tim_top">
     <collision>
       <origin xyz="0 0 0" rpy="0 0 0"/>
@@ -120,8 +120,8 @@
     </inertial>
   </link>
-  <joint name="neato_laser" type="fixed">
+  <joint name="tim_top" type="fixed">
     <origin xyz="0 0 ${lidarZPos}" rpy="3.14159 0 0"/>
     <parent link="chassis"/>
-    <child link="neato_laser"/>
+    <child link="tim_top"/>
   </joint>
   <xacro:caster_wheel name="caster_wheel_upper_right" tX="${chassisLength/2 - 0.03}" tY="${chassisWidth/2 - 0.03}" />

Commit message: update and create launch files for new krabi

File: urdf/krabby.xacro (robot description, xacro)
@@ -2,36 +2,19 @@
 <robot name="krabby"
   xmlns:xacro="http://www.ros.org/wiki/xacro">
-  <xacro:property name="PI" value="3.1415926535897931"/>
-  <xacro:property name="chassisHeight" value="0.005"/>
-  <xacro:property name="chassisLength" value="0.250"/>
-  <xacro:property name="chassisWidth" value="0.250"/>
-  <xacro:property name="chassisMass" value="2"/>
-  <xacro:property name="wheelWidth" value="0.008"/>
-  <xacro:property name="wheelRadius" value="0.032"/>
-  <xacro:property name="wheelXPos" value="0.08"/>
-  <xacro:property name="wheelMass" value="0.02"/>
-  <xacro:property name="casterWheelRadius" value="${wheelRadius/2-0.001}"/>
-  <xacro:property name="casterWheelMass" value="0.01"/>
-  <xacro:property name="cameraSize" value="0.05"/>
-  <xacro:property name="cameraMass" value="0.1"/>
-  <xacro:property name="lidarZPos" value="0.3"/>
-  <!-- mapping
-    <xacro:property name="lidarZPos" value="0.06"/>
-  -->
-  <xacro:property name="lidarMass" value="0.1"/>
-  <xacro:property name="lidarRadius" value="0.05"/>
-  <xacro:property name="lidarHeight" value="0.01"/>
-  <xacro:property name="arucoSize" value="0.1"/>
+  <xacro:include filename="properties.xacro"/>
+  <xacro:include filename="materials.xacro"/>
   <xacro:include filename="krabby.gazebo"/>
-  <xacro:include filename="materials.xacro"/>
   <xacro:include filename="macros.xacro"/>
   <link name="base_link"/>
+  <!-- ************************************************************** -->
+  <!-- chassis                                                        -->
+  <!-- ************************************************************** -->
   <joint name="base_joint" type="fixed">
     <parent link="base_link"/>
     <child link="chassis"/>
+    <origin xyz="0 0 ${chassisDistanceAuSol}" rpy="0 0 0"/>
   </joint>
   <link name='chassis'>
     <collision>
-      <origin xyz="0 0 ${wheelRadius}" rpy="0 0 0"/>
       <geometry>
         <box size="${chassisLength} ${chassisWidth} ${chassisHeight}"/>
@@ -39,5 +22,4 @@
     </collision>
     <visual>
-      <origin xyz="0 0 ${wheelRadius}" rpy="0 0 0"/>
       <geometry>
         <box size="${chassisLength} ${chassisWidth} ${chassisHeight}"/>
@@ -46,9 +28,79 @@
     </visual>
     <inertial>
-      <origin xyz="0 0 ${wheelRadius}" rpy="0 0 0"/>
       <mass value="${chassisMass}"/>
       <xacro:box_inertia m="${chassisMass}" x="${chassisLength}" y="${chassisWidth}" z="${chassisHeight}"/>
     </inertial>
   </link>
+  <!-- ************************************************************** -->
+  <!-- body                                                        -->
+  <!-- ************************************************************** -->
+  <joint name="body_joint" type="fixed">
+    <parent link="chassis"/>
+    <child link="body"/>
+    <origin xyz="${bodyOffsetX} ${bodyOffsetY} ${bodyOffsetZ}"/>
+  </joint>
+  <link name='body'>
+    <collision>
+      <geometry>
+        <box size="${bodyLength} ${bodyWidth} ${bodyHeight}"/>
+      </geometry>
+    </collision>
+    <visual>
+      <geometry>
+        <box size="${bodyLength} ${bodyWidth} ${bodyHeight}"/>
+      </geometry>
+      <material name="blue"/>
+    </visual>
+    <inertial>
+      <mass value="${bodyMass}"/>
+      <xacro:box_inertia m="${bodyMass}" x="${bodyLength}" y="${bodyWidth}" z="${bodyHeight}"/>
+    </inertial>
+  </link>
+  <!-- ************************************************************** -->
+  <!-- wheels                                                      -->
+  <!-- ************************************************************** -->
+  <xacro:wheel lr="left" parent="chassis" tX="${wheelXOffset}" tY="${wheelYOffset}" tZ="${wheelZOffset}"/>
+  <xacro:wheel lr="right" parent="chassis" tX="${wheelXOffset}" tY="${-wheelYOffset}" tZ="${wheelZOffset}"/>
+  <xacro:caster_wheel parent="chassis" name="caster_fr" tX="${casterXOffset}" tY="-${casterYOffset}"/>
+  <xacro:caster_wheel parent="chassis" name="caster_fl" tX="${casterXOffset}" tY="${casterYOffset}"/>
+  <xacro:caster_wheel parent="chassis" name="caster_rr" tX="-${casterXOffset}" tY="-${casterYOffset}"/>
+  <xacro:caster_wheel parent="chassis" name="caster_rl" tX="-${casterXOffset}" tY="${casterYOffset}"/>
+  <!-- ************************************************************** -->
+  <!-- lidar                                                           -->
+  <!-- ************************************************************** -->
+  <joint name="lidar_joint" type="fixed">
+    <parent link="body"/>
+    <child link="lidar"/>
+    <origin xyz="0 0 ${lidarZPos}"/>
+  </joint>
+  <link name='lidar'>
+    <inertial>
+      <mass value="${lidarMass}"/>
+      <xacro:cylinder_inertia m="${lidarMass}" r="${lidarRadius}" h="${lidarHeight}"/>
+    </inertial>
+    <!-- No collision on purpose, to not block lidar rays in simulation -->
+    <!-- <collision name="lidar_collision"> -->
+    <!--   <pose>0 0 0 0 0 0</pose> -->
+    <!--   <geometry> -->
+    <!--     <cylinder length="${lidarHeight}" radius="${lidarRadius}"/> -->
+    <!--   </geometry> -->
+    <!-- </collision> -->
+    <visual name="lidar_visual">
+      <pose>0 0 0 0 0 0</pose>
+      <geometry>
+        <cylinder length="${lidarHeight}" radius="${lidarRadius}"/>
+      </geometry>
+      <material name="black"/>
+    </visual>
+  </link>
+  <!-- ************************************************************** -->
+  <!-- camera                                                           -->
+  <!-- ************************************************************** -->
+  <!-- ************************************************************** -->
+  <!-- aruco                                                           -->
+  <!-- ************************************************************** -->
+  <!-- ************************************************************** -->
+  <!-- the following is optional, not corrected yet                    -->
+  <!-- ************************************************************** -->
   <link name="aruco_link">
     <inertial>
@@ -120,14 +172,8 @@
     </inertial>
   </link>
-  <joint name="tim_top" type="fixed">
+  <joint name="tim_top_joint" type="fixed">
     <origin xyz="0 0 ${lidarZPos}" rpy="3.14159 0 0"/>
     <parent link="chassis"/>
     <child link="tim_top"/>
   </joint>
-  <xacro:caster_wheel name="caster_wheel_upper_right" tX="${chassisLength/2 - 0.03}" tY="${chassisWidth/2 - 0.03}" />
-  <xacro:caster_wheel name="caster_wheel_upper_left" tX="${-(chassisLength/2 - 0.03)}" tY="${chassisWidth/2 - 0.03}" />
-  <xacro:caster_wheel name="caster_wheel_lower_right" tX="${chassisLength/2 - 0.03}" tY="${-(chassisWidth/2 - 0.03)}" />
-  <xacro:caster_wheel name="caster_wheel_lower_left" tX="${-(chassisLength/2 - 0.03)}" tY="${-(chassisWidth/2 - 0.03)}" />
-  <xacro:wheel lr="left" tY="${wheelXPos}"/>
-  <xacro:wheel lr="right" tY="${-wheelXPos}"/>
 </robot>

File: urdf/macros.xacro (robot description, xacro)
@@ -11,5 +11,5 @@
         <inertia ixx="${2*m*r*r/5}" ixy="0" ixz="0" iyy="${2*m*r*r/5}" iyz="0" izz="${2*m*r*r/5}" />
     </xacro:macro>
-    <xacro:macro name="wheel" params="lr tY">
+    <xacro:macro name="wheel" params="lr parent tX:=0 tY:=0 tZ:=0">
         <link name="${lr}_wheel">
             <collision>
@@ -44,7 +44,7 @@
         </gazebo>
         <joint name="${lr}_wheel_hinge" type="continuous">
-            <parent link="chassis"/>
+            <parent link="${parent}"/>
             <child link="${lr}_wheel"/>
-            <origin xyz="0 ${tY} ${wheelRadius}" rpy="0 0 0"/>
+            <origin xyz="${tX} ${tY} ${tZ}" rpy="0 0 0"/>
             <axis xyz="0 1 0" rpy="0 0 0"/>
             <limit effort="100" velocity="100"/>
@@ -62,8 +62,8 @@
         </transmission-->
     </xacro:macro>
-    <xacro:macro name="caster_wheel" params="name tX tY">
+    <xacro:macro name="caster_wheel" params="parent name tX tY">
         <link name="${name}">
             <collision>
-                <origin xyz="${tX} ${tY} ${casterWheelRadius}" rpy="0 0 0"/>
+                <origin xyz="${tX} ${tY} 0" rpy="0 0 0"/>
                 <geometry>
                     <sphere radius="${casterWheelRadius}"/>
@@ -71,5 +71,5 @@
             </collision>
             <visual>
-                <origin xyz="${tX} ${tY} ${casterWheelRadius}" rpy="0 0 0"/>
+                <origin xyz="${tX} ${tY} 0" rpy="0 0 0"/>
                 <geometry>
                     <sphere radius="${casterWheelRadius}"/>
@@ -83,6 +83,6 @@
             </inertial>
         </link>
-        <joint name="${name}" type="fixed">
-            <parent link="chassis"/>
+        <joint name="${name}_joint" type="fixed">
+            <parent link="${parent}"/>
             <child link="${name}"/>
         </joint>

Commit message: add 3d model (todo : fix position)

File: urdf/krabby.xacro (robot description, xacro)
@@ -46,7 +46,13 @@
       </geometry>
     </collision>
+    <!--Kraboss_base_assembly_For_Simu_v1.stl-->
     <visual>
       <geometry>
-        <box size="${bodyLength} ${bodyWidth} ${bodyHeight}"/>
+        <!--<origin xyz="0 ${chassisWidth}/2 ${chassisDistanceAuSol}" rpy="0 0 0"/>-->
+        <!--<mesh><uri>file://Kraboss_base_assembly_For_Simu_v1.stl</uri></mesh>-->
+        <!--<pose>0 ${chassisWidth}/2 0 0 -0 0</pose>-->
+        <mesh scale="0.001 0.001 0.001" filename="file://$(find krabby_description)/models/Kraboss_base_assembly_For_Simu_v1.stl"/>
+        <!--<mesh scale="0.001 0.001 0.001" filename="file://$(find krabby_description)/models/Kraboss_base_assembly_For_Simu_v1.dae"/>-->
+        <!--<box size="${bodyLength} ${bodyWidth} ${bodyHeight}"/>-->
       </geometry>
       <material name="blue"/>

Commit message: add ldlidar top

File: urdf/krabby.xacro (robot description, xacro)
@@ -158,5 +158,5 @@
     <child link="camera_link"/>
   </joint>
-  <link name="tim_top">
+  <link name="ldlidar_top">
     <collision>
       <origin xyz="0 0 0" rpy="0 0 0"/>
@@ -178,4 +178,29 @@
     </inertial>
   </link>
+  <joint name="ldlidar_top_joint" type="fixed">
+    <origin xyz="0 0 ${lidarZPos}" rpy="0 0 0"/>
+    <parent link="chassis"/>
+    <child link="ldlidar_top"/>
+  </joint>
+  <link name="tim_top">
+    <collision>
+      <origin xyz="0 0 0" rpy="0 0 0"/>
+      <geometry>
+        <cylinder length="${lidarHeight}" radius="${lidarRadius}"/>
+      </geometry>
+    </collision>
+    <visual>
+      <origin xyz="0 0 0" rpy="0 0 0"/>
+      <geometry>
+        <cylinder length="${lidarHeight}" radius="${lidarRadius}"/>
+      </geometry>
+      <material name="black"/>
+    </visual>
+    <inertial>
+      <origin xyz="0 0 0" rpy="0 0 0"/>
+      <mass value="${lidarMass}"/>
+      <xacro:cylinder_inertia m="${lidarMass}" r="${lidarRadius}" h="${lidarHeight}"/>
+    </inertial>
+  </link>
   <joint name="tim_top_joint" type="fixed">
     <origin xyz="0 0 ${lidarZPos}" rpy="3.14159 0 0"/>

Commit message: add missing Aruco

File: urdf/krabby.xacro (robot description, xacro)
@@ -124,5 +124,5 @@
       <pose>0 0 0 0 0 0</pose>
       <geometry>
-        <mesh filename="package://eurobot2020_gazebo/models/tag_aruco/meshes/tag_aruco.dae"/>
+        <mesh filename="models/tag_aruco/meshes/tag_aruco.dae"/>
       </geometry>
     </visual>

Commit message: fix previous commit

File: urdf/krabby.xacro (robot description, xacro)
@@ -124,5 +124,5 @@
       <pose>0 0 0 0 0 0</pose>
       <geometry>
-        <mesh filename="models/tag_aruco/meshes/tag_aruco.dae"/>
+        <mesh filename="file://$(find krabby_description)/models/tag_aruco/meshes/tag_aruco.dae"/>
       </geometry>
     </visual>

Commit message: WiP lidars

File: urdf/krabby.xacro (robot description, xacro)
@@ -41,9 +41,9 @@
   </joint>
   <link name='body'>
-    <collision>
+    <!--<collision>
       <geometry>
         <box size="${bodyLength} ${bodyWidth} ${bodyHeight}"/>
       </geometry>
-    </collision>
+    </collision>-->
     <!--Kraboss_base_assembly_For_Simu_v1.stl-->
     <visual>
@@ -73,10 +73,10 @@
   <xacro:caster_wheel parent="chassis" name="caster_rl" tX="-${casterXOffset}" tY="${casterYOffset}"/>
   <!-- ************************************************************** -->
-  <!-- lidar                                                           -->
+  <!-- lidar (exemple, not used)                                      -->
   <!-- ************************************************************** -->
   <joint name="lidar_joint" type="fixed">
     <parent link="body"/>
     <child link="lidar"/>
-    <origin xyz="0 0 ${lidarZPos}"/>
+    <origin xyz="0 0 ${lidarLD06_topZPos}"/>
   </joint>
   <link name='lidar'>
@@ -158,11 +158,15 @@
     <child link="camera_link"/>
   </joint>
+  <!-- ************************************************************** -->
+  <!-- lidar_top (LD06)                                               -->
+  <!-- ************************************************************** -->
   <link name="ldlidar_top">
-    <collision>
-      <origin xyz="0 0 0" rpy="0 0 0"/>
-      <geometry>
-        <cylinder length="${lidarHeight}" radius="${lidarRadius}"/>
-      </geometry>
-    </collision>
+    <!-- No collision on purpose, to not block lidar rays in simulation -->
+    <!--<collision>
+      <origin xyz="0 0 0" rpy="0 0 0"/>
+      <geometry>
+        <cylinder length="${lidarHeight}" radius="${lidarRadius}"/>
+      </geometry>
+    </collision>-->
     <visual>
       <origin xyz="0 0 0" rpy="0 0 0"/>
@@ -179,15 +183,19 @@
   </link>
   <joint name="ldlidar_top_joint" type="fixed">
-    <origin xyz="0 0 ${lidarZPos}" rpy="0 0 0"/>
+    <origin xyz="0 0 ${lidarLD06_topZPos}" rpy="0 0 0"/>
     <parent link="chassis"/>
     <child link="ldlidar_top"/>
   </joint>
-  <link name="tim_top">
-    <collision>
-      <origin xyz="0 0 0" rpy="0 0 0"/>
-      <geometry>
-        <cylinder length="${lidarHeight}" radius="${lidarRadius}"/>
-      </geometry>
-    </collision>
+  <!-- ************************************************************** -->
+  <!-- lidar_bottom (TIM) for localisation on borders                 -->
+  <!-- ************************************************************** -->
+  <link name="tim_lidar_bottom">
+    <!-- No collision on purpose, to not block lidar rays in simulation -->
+    <!--<collision>
+      <origin xyz="0 0 0" rpy="0 0 0"/>
+      <geometry>
+        <cylinder length="${lidarHeight}" radius="${lidarRadius}"/>
+      </geometry>
+    </collision>-->
     <visual>
       <origin xyz="0 0 0" rpy="0 0 0"/>
@@ -203,8 +211,8 @@
     </inertial>
   </link>
-  <joint name="tim_top_joint" type="fixed">
-    <origin xyz="0 0 ${lidarZPos}" rpy="3.14159 0 0"/>
-    <parent link="chassis"/>
-    <child link="tim_top"/>
+  <joint name="tim_lidar_bottom_joint" type="fixed">
+    <origin xyz="${lidarTIM_bottom_XPos} ${lidarTIM_bottom_YPos} ${lidarTIM_bottom_ZPos}" rpy="0 0 ${lidarTIM_bottom_Yaw}"/>
+    <parent link="chassis"/>
+    <child link="tim_lidar_bottom"/>
   </joint>
 </robot>

File: urdf/properties.xacro (robot description, xacro)
@@ -30,7 +30,11 @@
   <xacro:property name="casterWheelMass" value="0.01"/>
   <!-- lidar -->
-  <xacro:property name="lidarZPos" value="0.3"/>
+  <xacro:property name="lidarLD06_topZPos" value="0.38"/>
+  <xacro:property name="lidarTIM_bottom_XPos" value="-0.07"/>
+  <xacro:property name="lidarTIM_bottom_YPos" value="0.091"/>
+  <xacro:property name="lidarTIM_bottom_ZPos" value="0.06"/>
+  <xacro:property name="lidarTIM_bottom_Yaw" value="2.35619449"/>
   <xacro:property name="lidarMass" value="0.1"/>
-  <xacro:property name="lidarRadius" value="0.05"/>
+  <xacro:property name="lidarRadius" value="0.02"/>
   <xacro:property name="lidarHeight" value="0.01"/>
   <!-- camera -->

Commit message: fix lidar position

File: urdf/krabby.xacro (robot description, xacro)
@@ -76,5 +76,5 @@
   <!-- ************************************************************** -->
   <joint name="lidar_joint" type="fixed">
-    <parent link="body"/>
+    <parent link="chassis"/>
     <child link="lidar"/>
     <origin xyz="0 0 ${lidarLD06_topZPos}"/>

Commit message: krabby_description => krabi_description

File: urdf/krabby.xacro (robot description, xacro)
@@ -52,6 +52,6 @@
         <!--<mesh><uri>file://Kraboss_base_assembly_For_Simu_v1.stl</uri></mesh>-->
         <!--<pose>0 ${chassisWidth}/2 0 0 -0 0</pose>-->
-        <mesh scale="0.001 0.001 0.001" filename="file://$(find krabby_description)/models/Kraboss_base_assembly_For_Simu_v1.stl"/>
-        <!--<mesh scale="0.001 0.001 0.001" filename="file://$(find krabby_description)/models/Kraboss_base_assembly_For_Simu_v1.dae"/>-->
+        <mesh scale="0.001 0.001 0.001" filename="file://$(find krabi_description)/models/Kraboss_base_assembly_For_Simu_v1.stl"/>
+        <!--<mesh scale="0.001 0.001 0.001" filename="file://$(find krabi_description)/models/Kraboss_base_assembly_For_Simu_v1.dae"/>-->
         <!--<box size="${bodyLength} ${bodyWidth} ${bodyHeight}"/>-->
       </geometry>
@@ -124,5 +124,5 @@
       <pose>0 0 0 0 0 0</pose>
       <geometry>
-        <mesh filename="file://$(find krabby_description)/models/tag_aruco/meshes/tag_aruco.dae"/>
+        <mesh filename="file://$(find krabi_description)/models/tag_aruco/meshes/tag_aruco.dae"/>
       </geometry>
     </visual>

File: urdf/krabby_campi.xacro (robot description, xacro)
@@ -5,7 +5,7 @@
   <xacro:property name="cameraSize" value="0.05"/>
   <xacro:property name="cameraMass" value="0.1"/>
-  <xacro:include filename="$(find krabby_description)/urdf/krabby_campi.gazebo"/>
-  <xacro:include filename="$(find krabby_description)/urdf/materials.xacro"/>
-  <xacro:include filename="$(find krabby_description)/urdf/macros.xacro"/>
+  <xacro:include filename="$(find krabi_description)/urdf/krabby_campi.gazebo"/>
+  <xacro:include filename="$(find krabi_description)/urdf/materials.xacro"/>
+  <xacro:include filename="$(find krabi_description)/urdf/macros.xacro"/>
   <link name="camera_campi_link">
     <collision>

Commit message: 2026 camera position (approximate)

File: urdf/krabby.xacro (robot description, xacro)
@@ -154,5 +154,5 @@
   </link>
   <joint name="camera_joint" type="fixed">
-    <origin xyz="${-cameraSize+chassisLength/2} 0 ${cameraSize+wheelRadius+cameraSize/2}" rpy="0 0 0"/>
+    <origin xyz="0 ${chassisLength/2+0.05} 0.3" rpy="0 1.57 1.57"/>
     <parent link="chassis"/>
     <child link="camera_link"/>

Commit message: Adapt to KV2 new cam

File: urdf/krabby.xacro (robot description, xacro)
@@ -154,5 +154,5 @@
   </link>
   <joint name="camera_joint" type="fixed">
-    <origin xyz="0 ${chassisLength/2+0.05} 0.3" rpy="0 1.57 1.57"/>
+    <origin xyz="0 -${chassisLength/2+0.05} 0.3" rpy="0 1.57 -1.57"/>
     <parent link="chassis"/>
     <child link="camera_link"/>
