Commit message: add IMU

File: urdf/krabby.xacro (robot description, xacro)
@@ -216,3 +216,30 @@
     <child link="tim_lidar_bottom"/>
   </joint>
+  <!-- ************************************************************** -->
+  <!-- IMU                                                            -->
+  <!-- ************************************************************** -->
+  <link name="imu_link">
+        <visual>
+            <geometry>
+                <box size="0.1 0.1 0.1" />
+            </geometry>
+            <material name="Cyan">
+                <color rgba="0 1.0 1.0 1.0" />
+            </material>
+        </visual>
+        <collision>
+            <geometry>
+                <box size="0.1 0.1 0.1" />
+            </geometry>
+        </collision>
+        <inertial>
+            <mass value=".1" />
+            <inertia ixx="0.145833" ixy="0.0" ixz="0.0" iyy="0.145833" iyz="0.0" izz="0.125" />
+        </inertial>
+    </link>
+    <joint name="imu_joint" type="fixed">
+       <parent link="base_link" />
+       <child link="imu_link" />
+       <origin xyz="0 0 ${bodyHeight/2}" />
+   </joint>
 </robot>

Commit message: update Krabi 3D model+fix camera position

File: urdf/krabby.xacro (robot description, xacro)
@@ -52,5 +52,5 @@
         <!--<mesh><uri>file://Kraboss_base_assembly_For_Simu_v1.stl</uri></mesh>-->
         <!--<pose>0 ${chassisWidth}/2 0 0 -0 0</pose>-->
-        <mesh scale="0.001 0.001 0.001" filename="file://$(find krabi_description)/models/Kraboss_base_assembly_For_Simu_v1.stl"/>
+        <mesh scale="0.001 0.001 0.001" filename="file://$(find krabi_description)/models/Kraboss_base_assembly_For_Simu_2026_v2.stl"/>
         <!--<mesh scale="0.001 0.001 0.001" filename="file://$(find krabi_description)/models/Kraboss_base_assembly_For_Simu_v1.dae"/>-->
         <!--<box size="${bodyLength} ${bodyWidth} ${bodyHeight}"/>-->
@@ -154,5 +154,5 @@
   </link>
   <joint name="camera_joint" type="fixed">
-    <origin xyz="0 -${chassisLength/2+0.05} 0.3" rpy="0 1.57 -1.57"/>
+    <origin xyz="0 -${chassisLength/2+0.08} 0.25" rpy="0 1.57 -1.57"/>
     <parent link="chassis"/>
     <child link="camera_link"/>
