Commit message: center KV2's model

File: urdf/properties.xacro (robot description, xacro)
@@ -9,7 +9,7 @@
   <xacro:property name="chassisMass" value="3"/>
   <!-- body -->
-  <xacro:property name="bodyOffsetX" value="-0.020"/>
-  <xacro:property name="bodyOffsetY" value="0.000"/>
-  <xacro:property name="bodyOffsetZ" value="0.150"/>
+  <xacro:property name="bodyOffsetX" value="0.010"/>
+  <xacro:property name="bodyOffsetY" value="-0.085"/>
+  <xacro:property name="bodyOffsetZ" value="0.000"/>
   <xacro:property name="bodyLength" value="0.170"/>
   <xacro:property name="bodyWidth" value="0.230"/>

Commit message: adapt to KV2

File: urdf/properties.xacro (robot description, xacro)
@@ -19,5 +19,5 @@
   <xacro:property name="wheelWidth" value="0.008"/>
   <xacro:property name="wheelRadius" value="0.030"/>
-  <xacro:property name="wheelXOffset" value="-0.018"/>
+  <xacro:property name="wheelXOffset" value="-0.0"/>
   <xacro:property name="wheelYOffset" value="0.062"/>
   <xacro:property name="wheelZOffset" value="0.025"/>
